File: KICAD PROJECT/KICAD PROJECT.kicad_pcb (KiCad board)
At the start: 6 copper layers, 89.5 x 121.5 mm, 149 parts, among them IC1 TPS61032PWP, J1 AudioJack3_Ground_SwitchTR, J2 Conn_01x02_Pin, J4 Conn_01x08_Socket, J5 Conn_01x08_Socket, P1 USB_C_Plug_USB2.0, Q1 BC857, Q2 BSS84, Q3 BSS84, SW1 SW_Push, SW10 SW_Push, SW11 SW_Push, SW12 SW_Push, SW13 SW_Push, SW14 SW_Push, SW15 SW_Push, SW16 SW_Push, SW17 SW_Push, SW18 SW_Push, SW19 SW_Push, SW2 SW_Push, SW20 SW_Push, SW21 SW_Push, SW22 SW_Push, SW23 SW_Push, SW24 SW_Push, SW25 SW_Push, SW26 SW_Push, SW27 SW_Push, SW28 SW_Push, SW29 SW_Push, SW3 SW_Push, SW30 SW_Push, SW31 SW_Push, SW32 SW_Push, SW33 SW_Push, SW34 SW_Push, SW35 SW_Push, SW37 SW_Push, SW38 SW_Push, SW39 SW_Push, SW4 SW_Push, SW40 SW_Push, SW41 SW_Push, SW42 SW_Push, SW43 SW_Push, SW44 SW_SPDT, SW5 SW_Push, SW6 SW_Push, SW7 SW_Push, SW8 SW_Push, SW9 SW_Push, U1 PCM5102A, U2 Raspberry pi Zero 2 w, U3 RP2040-ZERO, U4 PAM8302AAD, U8 MCP73833-xxx-MF

Commit message: Updates and gerbers
Parts:
- added R16: 4.5k, Resistor_SMD:R_0603_1608Metric_Pad0.98x0.95mm_HandSolder, F.Cu at (50.3, 57.3)
- IC1: footprint Package_SO:HTSSOP-16-1EP_4.4x5mm_P0.65mm_EP3.4x5mm_Mask2.66x2.46mm_ThermalVias -> Package_SO:HTSSOP-16-1EP_4.4x5mm_P0.65mm_EP3.4x5mm_Mask2.66x2.46mm
- R1: value 1k -> 2K
- R2: value 1k -> 4.5k; moved to F.Cu
- moved R2 65.8 mm to (50.3, 52.8)
- moved R3 1.33 mm to (101.8, 93.6), turned to 90 degrees
- moved SW44 0.39 mm to (72.8, 161.5)
- moved D18 0.33 mm to (90.8, 132.0)
- moved D19 0.33 mm to (82.3, 132.0)
Connections:
- C21 pad 2: CPGND -> Net-(C21-Pad2)
- R15 pad 2: Net-(C20-Pad1) -> Net-(C21-Pad2)
- R2 pad 1: Net-(R2-Pad1) -> +5V
- R2 pad 2: Net-(R1-Pad2) -> SDA
- R3 pad 1: Net-(R2-Pad1) -> Net-(R1-Pad2)
- U8 pad 5: unconnected-(U8-V_{SS}-Pad5) -> CPGND
Routing:
- net +5V: track 12.0 -> 285.7 mm, vias 3 -> 5
- net SCLK: track 102.7 -> 158.0 mm, vias 1 -> 0
- net +3.3V: track 250.3 -> 197.0 mm
- net CPGND: track 65.4 -> 113.6 mm, vias 119 -> 118
- net VBUS: track 53.1 -> 72.0 mm
- net RXD0: track 95.0 -> 108.7 mm
- net SCL: track 101.9 -> 114.7 mm, vias 0 -> 4
- net ENABLE_BACKLIGHT: track 59.4 -> 49.4 mm
- net MISO: track 103.9 -> 113.8 mm, vias 1 -> 2
- net GPIO21: track 88.1 -> 78.4 mm
- net I2S LRCK: track 53.6 -> 44.0 mm
- net SDA: track 109.5 -> 118.7 mm, vias 1 -> 3
- net GPIO16: track 58.9 -> 65.3 mm, vias 0 -> 1
- net MOSI: track 104.7 -> 110.7 mm, vias 1 -> 2
- net Net-(U4-~{SD}): track 36.6 -> 31.4 mm
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- added copper zone on In2.Cu, net CPGND
- removed copper zone on In4.Cu, net +5V
- removed copper zone on In1.Cu, net CPGND
- removed copper zone on In4.Cu, net CPGND
Other:
- copper layers 6 -> 4
- board text added: "Istratie Stefan 2025"
- board text added: "[ARC] rev. 0"
